Commit message: A3 轴可能是错误的，这里更新了A3轴。

File: urdf/robot_V10.urdf (robot description, URDF)
Before this commit: robot robot_V10, 21 links, 20 joints
Joints:
- joint joint_platform_A3: axis 0.123089726472094 0.835234243611025 0.535940927282611 -> 0 0 1

Commit message: fix

File: urdf/robot_V10.urdf (robot description, URDF)
Before this commit: robot robot_V10, 21 links, 20 joints
Joints:
- joint joint_platform_A3: axis 0 0 1 -> 0 0 -1
