Commit message: fix

File: urdf/robot_V13.urdf (robot description, URDF)
Before this commit: robot robot_V13, 20 links, 19 joints
Links:
- added link World
Joints:
- added joint world_to_base: type fixed, parent World, child base_link, origin xyz=0 0 0 rpy=0 0 0

Commit message: fix

File: urdf/robot_V13.urdf (robot description, URDF)
Before this commit: robot robot_V13, 21 links, 20 joints
Links:
- removed link World
Joints:
- removed joint world_to_base
